File: Alpsterium-pcb.kicad_sch (KiCad schematic)
At the start: 257 parts, among them SW0 KEYSW, SW1 KEYSW, SW10 KEYSW, SW100 KEYSW, SW101 KEYSW, SW102 KEYSW, SW103 KEYSW, SW104 KEYSW, SW105 KEYSW, SW106 KEYSW, SW107 KEYSW, SW108 KEYSW, SW109 KEYSW, SW11 KEYSW, SW110 KEYSW, SW111 KEYSW, SW112 KEYSW, SW113 KEYSW, SW114 KEYSW, SW115 KEYSW, SW116 KEYSW, SW117 KEYSW, SW118 KEYSW, SW119 KEYSW, SW12 KEYSW, SW120 KEYSW, SW121 KEYSW, SW122 KEYSW, SW123 KEYSW, SW124 KEYSW, SW125 KEYSW, SW126 KEYSW, SW127 KEYSW, SW128 KEYSW, SW129 KEYSW, SW13 KEYSW, SW130 KEYSW, SW131 KEYSW, SW132 KEYSW, SW134 KEYSW, SW135 KEYSW, SW136 KEYSW, SW137 KEYSW, SW138 KEYSW, SW139 KEYSW, SW14 KEYSW, SW140 KEYSW, SW141 KEYSW, SW142 KEYSW, SW143 KEYSW, SW144 KEYSW, SW145 KEYSW, SW146 KEYSW, SW147 KEYSW, SW148 KEYSW, SW149 KEYSW, SW15 KEYSW, SW150 KEYSW, SW151 KEYSW, SW152 KEYSW, SW153 KEYSW, SW154 KEYSW, SW155 KEYSW, SW156 KEYSW, SW157 KEYSW, SW158 KEYSW, SW159 KEYSW, SW16 KEYSW, SW17 KEYSW, SW18 KEYSW, SW19 KEYSW, SW2 KEYSW, SW20 KEYSW, SW21 KEYSW, SW22 KEYSW, SW23 KEYSW, SW24 KEYSW, SW25 KEYSW, SW26 KEYSW, SW27 KEYSW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

Commit message: modified:   Alpsterium-pcb.dsn 	modified:   Alpsterium-pcb.kicad_pcb 	modified:   Alpsterium-pcb.kicad_sch 	modified:   fp-info-cache
Parts:
- added D51: D_Small, cftkb:D_DO-35_SOD27_P5.08mm_Horizontal, symbol Device:D_Small
- added SW133: KEYSW, MX_Alps_Hybrid:MX-1.5U-NoLED, symbol Alpsterium-pcb-rescue:KEYSW-keyboard_parts-mysterium-pcb-rescue
- SW111: footprint MX_Alps_Hybrid:MX-2.75U-ReversedStabilizers-NoLED -> MX_Alps_Hybrid:MX-2.25U-ReversedStabilizers-NoLED
- renumbered D90 to D87, D92 to D88, D93 to D89, D94 to D90, D97 to D91, D98 to D92, D142 to D93, D69 to DN1
Connections:
- net VBUS: now also D51.2 (A); no longer U1.40 (GND_or_5V)
- net col0: now also SW133.1
- net at D50.2 (A), SW50.2, SW51.2: now also SW133.2
- net at D91.2 (A), SW107.2, SW131.2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: no longer SW97.2
- net NA: no longer names the net of U1.6 (A9)
- new net VCC: D51.1 (K), U1.40 (GND_or_5V)
- no-connect marks 2 -> 12
