File: Alpsterium-pcb.kicad_pcb (KiCad board)
At the start: 2 copper layers, 347.7 x 146.6 mm, 257 parts, among them SW0 KEYSW, SW1 KEYSW, SW10 KEYSW, SW100 KEYSW, SW101 KEYSW, SW102 KEYSW, SW103 KEYSW, SW104 KEYSW, SW105 KEYSW, SW106 KEYSW, SW107 KEYSW, SW108 KEYSW, SW109 KEYSW, SW11 KEYSW, SW110 KEYSW, SW111 KEYSW, SW112 KEYSW, SW113 KEYSW, SW114 KEYSW, SW115 KEYSW, SW116 KEYSW, SW117 KEYSW, SW118 KEYSW, SW119 KEYSW, SW12 KEYSW, SW120 KEYSW, SW121 KEYSW, SW122 KEYSW, SW123 KEYSW, SW124 KEYSW, SW125 KEYSW, SW126 KEYSW, SW127 KEYSW, SW128 KEYSW, SW129 KEYSW, SW13 KEYSW, SW130 KEYSW, SW131 KEYSW, SW132 KEYSW, SW134 KEYSW, SW135 KEYSW, SW136 KEYSW, SW137 KEYSW, SW138 KEYSW, SW139 KEYSW, SW14 KEYSW, SW140 KEYSW, SW141 KEYSW, SW142 KEYSW, SW143 KEYSW, SW144 KEYSW, SW145 KEYSW, SW146 KEYSW, SW147 KEYSW, SW148 KEYSW, SW149 KEYSW, SW15 KEYSW, SW150 KEYSW, SW151 KEYSW, SW152 KEYSW, SW153 KEYSW, SW154 KEYSW, SW155 KEYSW, SW156 KEYSW, SW157 KEYSW, SW158 KEYSW, SW159 KEYSW, SW16 KEYSW, SW17 KEYSW, SW18 KEYSW, SW19 KEYSW, SW2 KEYSW, SW20 KEYSW, SW21 KEYSW, SW22 KEYSW, SW23 KEYSW, SW24 KEYSW, SW25 KEYSW, SW26 KEYSW, SW27 KEYSW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

Commit message: modified:   Alpsterium-pcb.dsn 	modified:   Alpsterium-pcb.kicad_pcb 	modified:   Alpsterium-pcb.kicad_sch 	modified:   fp-info-cache
Parts:
- added D51: D_Small, cftkb:D_DO-35_SOD27_P5.08mm_Horizontal, F.Cu at (230.1, 62.3)
- added SW133: KEYSW, MX_Alps_Hybrid:MX-1.5U-NoLED, F.Cu at (51.5, 153.9)
- SW111: footprint MX_Alps_Hybrid:MX-2.75U-ReversedStabilizers-NoLED -> MX_Alps_Hybrid:MX-2.25U-ReversedStabilizers-NoLED
- moved SW111 4.92 mm to (58.6, 173.1)
- renumbered D90 to D87, D92 to D88, D93 to D89, D94 to D90, D97 to D91, D98 to D92, D142 to D93, D69 to DN1
Connections:
- D91 pad 2: Net-(D97-A) -> Net-(D91-A)
- SW107 pad 2: Net-(D97-A) -> Net-(D91-A)
- SW131 pad 2: Net-(D97-A) -> Net-(D91-A)
- SW132 pad 2: Net-(D97-A) -> Net-(D91-A)
- SW97 pad 2: Net-(D97-A) -> unconnected-(SW97-Pad2)
- U1 pad 40: VBUS -> VCC
- U1 pad 6: NA -> unconnected-(U1-A9)
Routing:
- net GND: track 9.24 -> 159.5 mm, vias 18 -> 4
- net col9: track 238.5 -> 343.3 mm, vias 1 -> 5
- net Net-(D8-A): track 99.2 -> 0.00 mm, vias 2 -> 0
- net row0: track 488.0 -> 406.9 mm, vias 4 -> 3
- net Net-(D74-A): track 267.8 -> 190.3 mm, vias 2 -> 0
- net Net-(D97-A): track 71.3 -> 0.00 mm
- net Net-(D91-A): track 0.00 -> 69.5 mm
- net Net-(D1-A): track 41.7 -> 0.00 mm
- net row3: track 539.0 -> 497.6 mm, vias 12 -> 7
- net col2: track 387.5 -> 428.4 mm
- net Net-(D2-A): track 38.6 -> 0.00 mm
- net col3: track 346.0 -> 384.3 mm
- net col17: track 256.8 -> 225.8 mm, vias 1 -> 0
- net Net-(D29-A): track 91.6 -> 62.1 mm
- net col0: track 443.1 -> 413.9 mm
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- removed copper zone on B.Cu, net GND
- removed copper zone on F.Cu, net GND

Commit message: Add files via upload
Routing:
- net col4: track 366.5 -> 360.1 mm
- net GND: track 159.5 -> 153.7 mm
- net row0: track 406.9 -> 403.0 mm
- net Net-(D54-A): track 87.7 -> 84.1 mm
- net Net-(D80-A): track 103.6 -> 107.0 mm
- net Net-(D77-A): track 129.8 -> 131.6 mm
- net row2: track 383.8 -> 385.3 mm
- net Net-(D53-A): track 86.0 -> 87.5 mm
- net Net-(D46-A): track 152.0 -> 153.5 mm
- net col9: track 343.3 -> 342.1 mm
- net row3: track 497.6 -> 496.4 mm
- net Net-(DN1-A): track 157.2 -> 156.1 mm
- net Net-(D52-A): track 80.1 -> 81.1 mm
- net col0: track 413.9 -> 414.9 mm
- net col1: track 326.5 -> 327.5 mm
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